File: Esquema TK2000/tk2000/tk2000.kicad_sch (KiCad schematic)
At the start: 5 parts, among them U28 74LS244, U29 6502, U30 74LS245, U35 74LS244, U50 74LS138

Commit message: mais componentes no esquema
Parts:
- added U17: 74LS244, symbol 74xx:74LS244
- added U24, U8: 74LS273, symbol 74xx:74LS273
- added U51, U?: 74LS174, symbol 74xx:74LS174
- added U52: 74LS157, symbol 74xx:74LS157
- added U7: 74LS166, symbol 74xx:74LS166
- added U? (x2): 2764, Package_DIP:DIP-28_W15.24mm, symbol Memory_EPROM:2764
- added U?: 74LS194, symbol 74xx:74LS194
Connections:
- net Earth: no longer U50.8 (GND)
- net VCC: no longer U50.16 (VCC)
- net at U35.12 (O3a): now also U50.2 (A1)
- net at U35.7 (O1b): now also U50.1 (A0)
- net at U35.9 (O0b): now also U50.3 (A2)
- new net: U51.14 (D5), U7.13 (Qh)
- new net: U51.2 (Q0), U52.2 (I0a)
- new net: U51.7 (Q2), U52.3 (I1a)
- new net: U51.13 (D4), U51.15 (Q5), U52.5 (I0b)
- new net: U51.10 (Q3), U52.6 (I1b)
- new net: U51.1 (~{Mr}), U51.16 (VCC)
- new net: U51.11 (D3), U51.12 (Q4)
- new net: U51.5 (Q1), U51.6 (D2)
- new net GNDREF: U51.8 (GND), U52.15 (E), U52.8 (GND), U7.8 (GND), U8.10 (GND), U?.8 (GND)
Other:
- note added: "TECLADO"
- moved on the sheet: U50
